File: Hardware/Qwiic_Relay.brd (EAGLE design)
At the start: 25.4 x 57.1 mm, 60 parts, among them J4 AVR_SPI_PROG_3X2TESTPOINTS, K1 RELAY-SPDT, Q4 600mA/40V, U3 ATTINY85

Commit message: moving high voltage silk
Parts:
- moved U$26 1.80 mm to (11.4, 31.8)
Changed lines of the file:
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@@
 <element name="LOGO2" library="SparkFun-Aesthetics" package="REVISION" value="REVISION" x="-5.08" y="-11.43"/>
 <element name="U$10" library="SparkFun-Aesthetics" package="ORDERING_INSTRUCTIONS" value="" x="-34.29" y="-13.97"/>
-<element name="U$26" library="buzzard_labels (13)" package="WARNING#_HIGH_VOLTAGE0" value="" x="12.7" y="30.48" rot="MR270"/>
+<element name="U$26" library="buzzard_labels (13)" package="WARNING#_HIGH_VOLTAGE0" value="" x="11.43" y="31.75" rot="MR270"/>
 <element name="U$27" library="buzzard_labels (15)" package="HV2" value="" x="22.987" y="37.973" rot="MR270"/>
 <element name="U$28" library="buzzard_labels (15)" package="LV1" value="" x="22.987" y="43.053" rot="MR270"/>
